File: testDesign2/testDesign2.sch (KiCad schematic (older format))
At the start: 31 parts, among them SW1 SW_Push, U1 CC2640R2FRSM, Y1 32.768kHz, Y2 24MHz

Commit message: Enclosure and PCB needs to be a CIRCLE
Parts:
- SW1: footprint Button_Switch_SMD:SW_SPST_PTS810 -> testDesign:Switch_EVP-BB4A9B000
Connections:
- net ADC0: now also U1.24 (DIO_7); no longer U1.23 (DIO_6)
- net Button: now also U1.23 (DIO_6); no longer U1.24 (DIO_7)
- net GND: now also U1.33 (EGP)
Changed lines of the file:
@@
 F 0 "SW1" H 5300 2885 50  0000 C CNN
 F 1 "SW_Push" H 5300 2794 50  0000 C CNN
-F 2 "Button_Switch_SMD:SW_SPST_PTS810" H 5300 2800 50  0001 C CNN
+F 2 "testDesign:Switch_EVP-BB4A9B000" H 5300 2800 50  0001 C CNN
 F 3 "" H 5300 2800 50  0001 C CNN
 	1    5300 2600
@@
 Wire Wire Line
 	5600 2600 5600 2700
-Text GLabel 5450 4500 2    50   Input ~ 0
+Text GLabel 5450 4650 2    50   Input ~ 0
 Button
 Text GLabel 5000 2600 0    50   Input ~ 0
@@
 Wire Wire Line
 	6300 2900 6300 3000
-Text GLabel 5450 4650 2    50   Input ~ 0
+Text GLabel 5450 4500 2    50   Input ~ 0
 ADC0
 $Comp
@@
 NoConn ~ 3650 5950
 NoConn ~ 2950 5550
+Text GLabel 3500 4050 1    50   Input ~ 0
+GND
 $EndSCHEMATC

Commit message: Think PCB design is finished. Need to do last checkthrough.
Parts:
- C12, C13, C9: footprint Capacitor_SMD:C_0402_1005Metric -> Capacitor_SMD:C_0603_1608Metric
- TH1: footprint Resistor_THT:R_Axial_DIN0207_L6.3mm_D2.5mm_P2.54mm_Vertical -> Resistor_THT:R_Axial_DIN0204_L3.6mm_D1.6mm_P1.90mm_Vertical
Changed lines of the file:
@@
 F 0 "C9" H 3815 1296 50  0000 L CNN
 F 1 "10uF" H 3815 1205 50  0000 L CNN
-F 2 "Capacitor_SMD:C_0402_1005Metric" H 3738 1100 50  0001 C CNN
+F 2 "Capacitor_SMD:C_0603_1608Metric" H 3738 1100 50  0001 C CNN
 F 3 "~" H 3700 1250 50  0001 C CNN
 	1    3700 1250
@@
 F 0 "C12" H 4315 1296 50  0000 L CNN
 F 1 "100nF" H 4315 1205 50  0000 L CNN
-F 2 "Capacitor_SMD:C_0402_1005Metric" H 4238 1100 50  0001 C CNN
+F 2 "Capacitor_SMD:C_0603_1608Metric" H 4238 1100 50  0001 C CNN
 F 3 "~" H 4200 1250 50  0001 C CNN
 	1    4200 1250
@@
 Wire Wire Line
 	4100 5950 4100 6350
-$Comp
-L testDesign2-rescue:GND-power #PWR01
-U 1 1 5C9740CF
-P 1250 1500
-F 0 "#PWR01" H 1250 1250 50  0001 C CNN
-F 1 "GND" H 1255 1327 50  0000 C CNN
-F 2 "" H 1250 1500 50  0001 C CNN
-F 3 "" H 1250 1500 50  0001 C CNN
-	1    1250 1500
-	1    0    0    -1
-$EndComp
 Wire Wire Line
 	1250 1200 1250 1350
 Wire Wire Line
 	1000 1350 1250 1350
-Connection ~ 1250 1350
-Wire Wire Line
-	1250 1350 1250 1500
 $Comp
 L testDesign2-rescue:TestPoint-Connector TP5
@@
 	7250 1400 7250 1500
 Wire Wire Line
-	6750 1100 6350 1100
+	6750 1100 6500 1100
 Wire Wire Line
 	6350 1100 6350 950
@@
 F 0 "C13" H 6115 1296 50  0000 L CNN
 F 1 "10uF" H 6115 1205 50  0000 L CNN
-F 2 "Capacitor_SMD:C_0402_1005Metric" H 6038 1100 50  0001 C CNN
+F 2 "Capacitor_SMD:C_0603_1608Metric" H 6038 1100 50  0001 C CNN
 F 3 "~" H 6000 1250 50  0001 C CNN
 	1    6000 1250
@@
 F 0 "TH1" H 6405 2646 50  0000 L CNN
 F 1 "Thermistor" H 6405 2555 50  0000 L CNN
-F 2 "Resistor_THT:R_Axial_DIN0207_L6.3mm_D2.5mm_P2.54mm_Vertical" H 6300 2600 50  0001 C CNN
+F 2 "Resistor_THT:R_Axial_DIN0204_L3.6mm_D1.6mm_P1.90mm_Vertical" H 6300 2600 50  0001 C CNN
 F 3 "~" H 6300 2600 50  0001 C CNN
 	1    6300 2600
@@
 Text GLabel 3500 4050 1    50   Input ~ 0
 GND
+Connection ~ 1250 1350
+Wire Wire Line
+	1250 1350 1250 1500
+$Comp
+L testDesign2-rescue:GND-power #PWR0101
+U 1 1 5C9B37A4
+P 1250 1500
+F 0 "#PWR0101" H 1250 1250 50  0001 C CNN
+F 1 "GND" H 1255 1327 50  0000 C CNN
+F 2 "" H 1250 1500 50  0001 C CNN
+F 3 "" H 1250 1500 50  0001 C CNN
+	1    1250 1500
+	1    0    0    -1
+$EndComp
+$Comp
+L power:PWR_FLAG #FLG0101
+U 1 1 5C9ADA95
+P 1250 1350
+F 0 "#FLG0101" H 1250 1425 50  0001 C CNN
+F 1 "PWR_FLAG" V 1250 1478 50  0000 L CNN
+F 2 "" H 1250 1350 50  0001 C CNN
+F 3 "~" H 1250 1350 50  0001 C CNN
+	1    1250 1350
+	0    1    1    0
+$EndComp
+$Comp
+L power:PWR_FLAG #FLG0102
+U 1 1 5C9ADB80
+P 2300 1100
+F 0 "#FLG0102" H 2300 1175 50  0001 C CNN
+F 1 "PWR_FLAG" H 2300 1273 50  0000 C CNN
+F 2 "" H 2300 1100 50  0001 C CNN
+F 3 "~" H 2300 1100 50  0001 C CNN
+	1    2300 1100
+	-1   0    0    1
+$EndComp
+Connection ~ 2300 1100
+$Comp
+L power:PWR_FLAG #FLG0103
+U 1 1 5C9AE24A
+P 6500 1100
+F 0 "#FLG0103" H 6500 1175 50  0001 C CNN
+F 1 "PWR_FLAG" H 6500 1273 50  0000 C CNN
+F 2 "" H 6500 1100 50  0001 C CNN
+F 3 "~" H 6500 1100 50  0001 C CNN
+	1    6500 1100
+	-1   0    0    1
+$EndComp
+Connection ~ 6500 1100
+Wire Wire Line
+	6500 1100 6350 1100
 $EndSCHEMATC

Commit message: Added mounts to PCB and started enclosure.
Parts:
- added H1: MountingHole, testDesign:MountingHole_1.2mm_M1, symbol Mechanical:MountingHole
Changed lines of the file:
@@
 Wire Wire Line
 	6500 1100 6350 1100
+$Comp
+L Mechanical:MountingHole H1
+U 1 1 5C9AE16C
+P 1000 2300
+F 0 "H1" H 1100 2346 50  0000 L CNN
+F 1 "MountingHole" H 1100 2255 50  0000 L CNN
+F 2 "testDesign:MountingHole_1.2mm_M1" H 1000 2300 50  0001 C CNN
+F 3 "~" H 1000 2300 50  0001 C CNN
+	1    1000 2300
+	1    0    0    -1
+$EndComp
 $EndSCHEMATC

Commit message: Recovered correct testDesign files from old stash
Parts:
- added TP1, TP2, TP3: TP, TestPoint:TestPoint_Pad_D1.0mm, symbol testDesign2-rescue:TestPoint-Connector
Connections:
- net GND: now also TP3.1
- net at U1.10 (DIO_2): now also TP2.1
- net at U1.9 (DIO_1): now also TP1.1
- no-connect marks 7 -> 5
Changed lines of the file:
@@
 NoConn ~ 4700 4050
 NoConn ~ 5450 4800
-NoConn ~ 3800 5950
-NoConn ~ 3650 5950
 NoConn ~ 2950 5550
 Text GLabel 3500 4050 1    50   Input ~ 0
@@
 	1    0    0    -1
 $EndComp
+$Comp
+L testDesign2-rescue:TestPoint-Connector TP1
+U 1 1 5CB567D6
+P 3650 5950
+F 0 "TP1" H 3700 6200 50  0000 R CNN
+F 1 "TP" H 3700 6300 50  0000 R CNN
+F 2 "TestPoint:TestPoint_Pad_D1.0mm" H 3850 5950 50  0001 C CNN
+F 3 "~" H 3850 5950 50  0001 C CNN
+	1    3650 5950
+	-1   0    0    1
+$EndComp
+$Comp
+L testDesign2-rescue:TestPoint-Connector TP2
+U 1 1 5CB56840
+P 3800 5950
+F 0 "TP2" H 3850 6200 50  0000 R CNN
+F 1 "TP" H 3850 6300 50  0000 R CNN
+F 2 "TestPoint:TestPoint_Pad_D1.0mm" H 4000 5950 50  0001 C CNN
+F 3 "~" H 4000 5950 50  0001 C CNN
+	1    3800 5950
+	-1   0    0    1
+$EndComp
+$Comp
+L testDesign2-rescue:TestPoint-Connector TP3
+U 1 1 5CB56C13
+P 1750 2650
+F 0 "TP3" H 1800 2900 50  0000 R CNN
+F 1 "TP" H 1800 3000 50  0000 R CNN
+F 2 "TestPoint:TestPoint_Pad_D1.0mm" H 1950 2650 50  0001 C CNN
+F 3 "~" H 1950 2650 50  0001 C CNN
+	1    1750 2650
+	-1   0    0    1
+$EndComp
+$Comp
+L testDesign2-rescue:GND-power #PWR0102
+U 1 1 5CB56D92
+P 1600 2650
+F 0 "#PWR0102" H 1600 2400 50  0001 C CNN
+F 1 "GND" H 1605 2477 50  0000 C CNN
+F 2 "" H 1600 2650 50  0001 C CNN
+F 3 "" H 1600 2650 50  0001 C CNN
+	1    1600 2650
+	1    0    0    -1
+$EndComp
+Wire Wire Line
+	1600 2650 1750 2650
 $EndSCHEMATC
